File: FirstTKLKB.sch (KiCad schematic (older format))
At the start: 19 parts, among them SW1 SW_Push, U1 ATmega32U4-AU, Y1 16MHz

Commit message: Position switch matrix
Parts:
- added J1: AVR-ISP-6, random-keyboard-parts:Reset_Pretty-Mask, symbol Connector:AVR-ISP-6
- added Q1: Q_NPN_BCE, Package_TO_SOT_SMD:SOT-223-3_TabPin2, symbol Device:Q_NPN_BCE
- added RC7: 1.5k, Resistor_SMD:R_0805_2012Metric_Pad1.15x1.40mm_HandSolder, symbol Device:R_Small
- C1, C2, C3, C4, C5, C6, C7, C8: footprint (none) -> Capacitor_SMD:C_0805_2012Metric_Pad1.15x1.40mm_HandSolder
- D1: footprint (none) -> LED_SMD:LED_0805_2012Metric_Pad1.15x1.40mm_HandSolder
- F1: value Power Polyfuse -> 500mA; footprint (none) -> Fuse:Fuse_0805_2012Metric_Pad1.15x1.40mm_HandSolder
- RC1: renamed from R1; footprint (none) -> Resistor_SMD:R_0805_2012Metric_Pad1.15x1.40mm_HandSolder
- RC2: renamed from R2; footprint (none) -> Resistor_SMD:R_0805_2012Metric_Pad1.15x1.40mm_HandSolder
- RC3: renamed from R3; footprint (none) -> Resistor_SMD:R_0805_2012Metric_Pad1.15x1.40mm_HandSolder
- RC4: renamed from R4; footprint (none) -> Resistor_SMD:R_0805_2012Metric_Pad1.15x1.40mm_HandSolder
- RC5: renamed from R5; footprint (none) -> Resistor_SMD:R_0805_2012Metric_Pad1.15x1.40mm_HandSolder
- SW1: footprint (none) -> random-keyboard-parts:SKQG-1155865
- USB1: footprint (none) -> random-keyboard-parts:Molex-0548190589
- Y1: footprint (none) -> Crystal:Crystal_SMD_3225-4Pin_3.2x2.5mm_HandSoldering
Connections:
- net GND: now also Q1.3 (E)
- net RESET: now reaches RC1.2, SW1.2, U1.13 (~RESET)
- net RESET: now also J1.5 (~RST)
- new net: Q1.1 (B), RC7.1
- new net LED_GND: Q1.2 (C)
Changed lines of the file:
@@
 F 0 "Y1" V 1650 2300 50  0000 L CNN
 F 1 "16MHz" V 1750 2300 50  0000 L CNN
-F 2 "" H 1700 2150 50  0001 C CNN
+F 2 "Crystal:Crystal_SMD_3225-4Pin_3.2x2.5mm_HandSoldering" H 1700 2150 50  0001 C CNN
 F 3 "~" H 1700 2150 50  0001 C CNN
 	1    1700 2150
@@
 F 0 "USB1" V 6637 2067 60  0000 C CNN
 F 1 "Molex-0548190589" V 6531 2067 60  0000 C CNN
-F 2 "" H 6100 2100 60  0001 C CNN
+F 2 "random-keyboard-parts:Molex-0548190589" H 6100 2100 60  0001 C CNN
 F 3 "" H 6100 2100 60  0001 C CNN
 	1    6100 2100
@@
 F 0 "C3" H 2042 3546 50  0000 L CNN
 F 1 "1uF" H 2042 3455 50  0000 L CNN
-F 2 "" H 1950 3500 50  0001 C CNN
+F 2 "Capacitor_SMD:C_0805_2012Metric_Pad1.15x1.40mm_HandSolder" H 1950 3500 50  0001 C CNN
 F 3 "~" H 1950 3500 50  0001 C CNN
 	1    1950 3500
@@
 F 0 "C2" V 1500 2200 50  0000 C CNN
 F 1 "22pF" V 1600 2250 50  0000 C CNN
-F 2 "" H 1400 2250 50  0001 C CNN
+F 2 "Capacitor_SMD:C_0805_2012Metric_Pad1.15x1.40mm_HandSolder" H 1400 2250 50  0001 C CNN
 F 3 "~" H 1400 2250 50  0001 C CNN
 	1    1400 2250
@@
 F 0 "C1" V 1629 2050 50  0000 C CNN
 F 1 "22pF" V 1538 2050 50  0000 C CNN
-F 2 "" H 1400 2050 50  0001 C CNN
+F 2 "Capacitor_SMD:C_0805_2012Metric_Pad1.15x1.40mm_HandSolder" H 1400 2050 50  0001 C CNN
 F 3 "~" H 1400 2050 50  0001 C CNN
 	1    1400 2050
@@
 	1600 2400 1600 2450
 $Comp
-L Device:R_Small R1
+L Device:R_Small RC1
 U 1 1 5EA025D7
 P 2000 1650
-F 0 "R1" H 2059 1696 50  0000 L CNN
+F 0 "RC1" H 2059 1696 50  0000 L CNN
 F 1 "10k" H 2059 1605 50  0000 L CNN
-F 2 "" H 2000 1650 50  0001 C CNN
+F 2 "Resistor_SMD:R_0805_2012Metric_Pad1.15x1.40mm_HandSolder" H 2000 1650 50  0001 C CNN
 F 3 "~" H 2000 1650 50  0001 C CNN
 	1    2000 1650
@@
 F 0 "SW1" H 1800 2135 50  0000 C CNN
 F 1 "SW_Push" H 1800 2044 50  0000 C CNN
-F 2 "" H 1800 2050 50  0001 C CNN
+F 2 "random-keyboard-parts:SKQG-1155865" H 1800 2050 50  0001 C CNN
 F 3 "~" H 1800 2050 50  0001 C CNN
 	1    1800 1850
@@
 P 7150 1900
 F 0 "F1" V 6945 1900 50  0000 C CNN
-F 1 "Power Polyfuse" V 7036 1900 50  0000 C CNN
-F 2 "" H 7200 1700 50  0001 L CNN
+F 1 "500mA" V 7036 1900 50  0000 C CNN
+F 2 "Fuse:Fuse_0805_2012Metric_Pad1.15x1.40mm_HandSolder" H 7200 1700 50  0001 L CNN
 F 3 "~" H 7150 1900 50  0001 C CNN
 	1    7150 1900
@@
 F 0 "D1" V 6896 2132 50  0000 R CNN
 F 1 "Power" V 6805 2132 50  0000 R CNN
-F 2 "" V 6850 2200 50  0001 C CNN
+F 2 "LED_SMD:LED_0805_2012Metric_Pad1.15x1.40mm_HandSolder" V 6850 2200 50  0001 C CNN
 F 3 "~" V 6850 2200 50  0001 C CNN
 	1    6850 2200
@@
 $EndComp
 $Comp
-L Device:R_Small R3
+L Device:R_Small RC3
 U 1 1 5EA2F552
 P 6850 2500
-F 0 "R3" H 6909 2546 50  0000 L CNN
+F 0 "RC3" H 6909 2546 50  0000 L CNN
 F 1 "220" H 6909 2455 50  0000 L CNN
-F 2 "" H 6850 2500 50  0001 C CNN
+F 2 "Resistor_SMD:R_0805_2012Metric_Pad1.15x1.40mm_HandSolder" H 6850 2500 50  0001 C CNN
 F 3 "~" H 6850 2500 50  0001 C CNN
 	1    6850 2500
@@
 $EndComp
 $Comp
-L Device:R_Small R2
+L Device:R_Small RC2
 U 1 1 5EA3D72F
 P 4000 3950
-F 0 "R2" V 3804 3950 50  0000 C CNN
+F 0 "RC2" V 3804 3950 50  0000 C CNN
 F 1 "10k" V 3895 3950 50  0000 C CNN
-F 2 "" H 4000 3950 50  0001 C CNN
+F 2 "Resistor_SMD:R_0805_2012Metric_Pad1.15x1.40mm_HandSolder" H 4000 3950 50  0001 C CNN
 F 3 "~" H 4000 3950 50  0001 C CNN
 	1    4000 3950
@@
 	6850 2600 6850 2750
 $Comp
-L Device:R_Small R5
+L Device:R_Small RC5
 U 1 1 5E9AB303
 P 1850 2850
-F 0 "R5" V 1550 3150 50  0000 C CNN
+F 0 "RC5" V 1550 3150 50  0000 C CNN
 F 1 "22" V 1650 3150 50  0000 C CNN
-F 2 "" H 1850 2850 50  0001 C CNN
+F 2 "Resistor_SMD:R_0805_2012Metric_Pad1.15x1.40mm_HandSolder" H 1850 2850 50  0001 C CNN
 F 3 "~" H 1850 2850 50  0001 C CNN
 	1    1850 2850
@@
 $EndComp
 $Comp
-L Device:R_Small R4
+L Device:R_Small RC4
 U 1 1 5E9AB7A6
 P 1550 2950
-F 0 "R4" V 1300 3250 50  0000 C CNN
+F 0 "RC4" V 1300 3250 50  0000 C CNN
 F 1 "22" V 1400 3250 50  0000 C CNN
-F 2 "" H 1550 2950 50  0001 C CNN
+F 2 "Resistor_SMD:R_0805_2012Metric_Pad1.15x1.40mm_HandSolder" H 1550 2950 50  0001 C CNN
 F 3 "~" H 1550 2950 50  0001 C CNN
 	1    1550 2950
@@
 F 0 "C5" H 8542 2696 50  0000 L CNN
 F 1 "0.1uF" H 8542 2605 50  0000 L CNN
-F 2 "" H 8450 2650 50  0001 C CNN
+F 2 "Capacitor_SMD:C_0805_2012Metric_Pad1.15x1.40mm_HandSolder" H 8450 2650 50  0001 C CNN
 F 3 "~" H 8450 2650 50  0001 C CNN
 	1    8450 2650
@@
 F 0 "C4" H 8142 2696 50  0000 L CNN
 F 1 "0.1uF" H 8142 2605 50  0000 L CNN
-F 2 "" H 8050 2650 50  0001 C CNN
+F 2 "Capacitor_SMD:C_0805_2012Metric_Pad1.15x1.40mm_HandSolder" H 8050 2650 50  0001 C CNN
 F 3 "~" H 8050 2650 50  0001 C CNN
 	1    8050 2650
@@
 F 0 "C6" H 8942 2696 50  0000 L CNN
 F 1 "0.1uF" H 8942 2605 50  0000 L CNN
-F 2 "" H 8850 2650 50  0001 C CNN
+F 2 "Capacitor_SMD:C_0805_2012Metric_Pad1.15x1.40mm_HandSolder" H 8850 2650 50  0001 C CNN
 F 3 "~" H 8850 2650 50  0001 C CNN
 	1    8850 2650
@@
 F 0 "C7" H 9342 2696 50  0000 L CNN
 F 1 "10uF" H 9342 2605 50  0000 L CNN
-F 2 "" H 9250 2650 50  0001 C CNN
+F 2 "Capacitor_SMD:C_0805_2012Metric_Pad1.15x1.40mm_HandSolder" H 9250 2650 50  0001 C CNN
 F 3 "~" H 9250 2650 50  0001 C CNN
 	1    9250 2650
@@
 F 0 "C8" H 9692 2696 50  0000 L CNN
 F 1 "47uF" H 9692 2605 50  0000 L CNN
-F 2 "" H 9600 2650 50  0001 C CNN
+F 2 "Capacitor_SMD:C_0805_2012Metric_Pad1.15x1.40mm_HandSolder" H 9600 2650 50  0001 C CNN
 F 3 "~" H 9600 2650 50  0001 C CNN
 	1    9600 2650
@@
 	9600 2750 9250 2750
 Connection ~ 9250 2750
+$Comp
+L Connector:AVR-ISP-6 J1
+U 1 1 5EB2BF5B
+P 8400 4250
+F 0 "J1" H 8071 4346 50  0000 R CNN
+F 1 "AVR-ISP-6" H 8071 4255 50  0000 R CNN
+F 2 "random-keyboard-parts:Reset_Pretty-Mask" V 8150 4300 50  0001 C CNN
+F 3 " ~" H 7125 3700 50  0001 C CNN
+	1    8400 4250
+	1    0    0    -1
+$EndComp
+Text GLabel 2150 1200 0    50   Input ~ 0
+RESET
+Wire Wire Line
+	2150 1200 2150 1850
+Connection ~ 2150 1850
+Text GLabel 8800 4350 2    50   Input ~ 0
+RESET
+$Comp
+L Device:Q_NPN_BCE Q1
+U 1 1 5EB34BA8
+P 6750 5350
+F 0 "Q1" H 6941 5396 50  0000 L CNN
+F 1 "Q_NPN_BCE" H 6941 5305 50  0000 L CNN
+F 2 "Package_TO_SOT_SMD:SOT-223-3_TabPin2" H 6950 5450 50  0001 C CNN
+F 3 "~" H 6750 5350 50  0001 C CNN
+	1    6750 5350
+	1    0    0    -1
+$EndComp
+$Comp
+L power:GND #PWR014
+U 1 1 5EBE90E8
+P 6850 5800
+F 0 "#PWR014" H 6850 5550 50  0001 C CNN
+F 1 "GND" H 6855 5627 50  0000 C CNN
+F 2 "" H 6850 5800 50  0001 C CNN
+F 3 "" H 6850 5800 50  0001 C CNN
+	1    6850 5800
+	1    0    0    -1
+$EndComp
+Wire Wire Line
+	6850 5800 6850 5550
+Text GLabel 6850 4800 2    50   Input ~ 0
+LED_GND
+Wire Wire Line
+	6850 4800 6850 5150
+$Comp
+L Device:R_Small RC7
+U 1 1 5EBEBB54
+P 6100 5350
+F 0 "RC7" V 5904 5350 50  0000 C CNN
+F 1 "1.5k" V 5995 5350 50  0000 C CNN
+F 2 "Resistor_SMD:R_0805_2012Metric_Pad1.15x1.40mm_HandSolder" H 6100 5350 50  0001 C CNN
+F 3 "~" H 6100 5350 50  0001 C CNN
+	1    6100 5350
+	0    1    1    0
+$EndComp
+Wire Wire Line
+	6550 5350 6200 5350
 $EndSCHEMATC
